File: NodeMCU-Lora-Gateway.brd (EAGLE design)
At the start: 59.7 x 40.6 mm, 31 parts, among them IC1 ATSHA204A, J2 GROVE-I2C, J3 Lipo Battery, J4 GROVE-I2C, J5 CON_HEADER_1X08-PTH, P1 PADSMALL, P2 PADNORMAL, Q1 BSS84, U1 RFM9x

Commit message: Bump to V1.3 version
* SMA/UFL Antenna connector has been size reduced
* Antenna trace and RF Module surrounded with via for better RF
isolation
* Increased "Isolate" ground planes to avoid shorts between connectors
and ground (may happen sometimes after soldering)
* I2C OLED connector is now "lock" version, you can just plug to test it
will fit without connector
* No more LED solder pad to choose VIN/3V3, added 1N4148 diode from 5V
for the 1st LED to decrease VCC to 4.4V, always works
* LORA version, added Microchip 64 bits Unique ID footprint 24AA02E64
* LORA version, done a diode logic OR for DIO0/DIO1/DIO2 for current
LIMC implementation
Parts:
- removed P1: PADSMALL, SteveMarple:PAD-SMALL
- removed SJLED: (no value), SparkFun-Passives:PAD-JUMPER-3-2OF3_NC_BY_TRACE_YES_SILK_LARGE
- removed U-FL: (no value), microbuilder:U.FL
- added C4: 100nF, _c2h:0805-CAP
- added D0, D1, D2, D5: 1N4148, Seeed-Discrete:SOD123-2.7X1.6
- added IC2: 24AA02E64, Microchip-24AA02E64T:SOT95P270X145-5N
- I2C_OLED: value CON_HEADER_1X04'SMALL'' -> CON_HEADER_1X04'LOCK'; device _c2h:M1X4 -> _c2h:1X04_LOCK
- J$1: value SMA_EDGE -> ANTENNATINY; device SparkFun-Connectors:SMA-EDGE -> _c2h:SMA_UFL_PAD_TINY
- moved I2C_OLED 5.27 mm to (38.1, 5.33)
- moved R1 5.08 mm to (21.6, 3.81)
- moved R2 4.45 mm to (24.8, 3.81)
- moved J$1 3.82 mm to (0.13, 5.21), turned to 180 degrees
- moved C2 0.63 mm to (50.2, 3.17)
Connections:
- new net DIO0: D0.1, U$3.DIO0, U1.DIO0
- new net DIO1: D1.1, U1.DIO1
- new net DIO2: D2.1, U1.DIO2
- net 3V3: now also C4.2, IC2.4; no longer SJLED.3
- net ANT: now also J$1.ANT1, J$1.ANT2, J$1.ANT3; no longer J$1.SIG, P1.1, U-FL.3
- net GND: now also C4.1, IC2.2, J$1.GND1, J$1.GND2, J$1.GND3, J$1.GND4; no longer J$1.GND@0, J$1.GND@1, J$1.GND@2, J$1.GND@3, U-FL.1, U-FL.2
- net RST: now also U1.RST
- net SCL: now also IC2.1
- net SDA: now also IC2.3
- net SS: now also D0.2, D1.2, D2.2; no longer U$3.DIO0, U1.DIO0
- net VIN: now also C3.2, D5.1, WS2812-1.2; no longer SJLED.1
- net VLED: now also D5.2; no longer C3.2, SJLED.2, WS2812-1.2
Routing:
- net DIO0: track 0.00 -> 43.2 mm, vias 0 -> 1
- net VLED: track 45.8 -> 9.81 mm, vias 2 -> 0
- net RST: track 59.9 -> 79.9 mm, vias 2 -> 4
- net SS: track 50.1 -> 35.9 mm, vias 0 -> 3
- net VIN: track 85.3 -> 99.1 mm
- net DIO1: track 0.00 -> 10.6 mm
- net 3V3: track 182.4 -> 174.3 mm
- net SDA: track 119.2 -> 124.3 mm
- net DIO2: track 0.00 -> 4.79 mm
- net SCL: track 136.8 -> 139.7 mm, vias 1 -> 2
- net ANT: track 20.4 -> 18.5 mm
- net N$1: track 13.6 -> 12.5 mm
- net GPIO0: track 111.8 -> 110.9 mm
- net DIN-2: track 34.8 -> 35.3 mm
Other:
- board text added: "NodeMCU Lora V1.3 http://hallard.me"
- board text added: "RF Antenna"
- board text removed: "NodeMCU Gateway V1.2 http://hallard.me"
- board text removed: "NodeMCU Lora Gateway V1.2 http://hallard.me"
- board text removed: "RF Ant"
- board text removed: "SMA"
- board text removed: "VIN <=5V"
- board text removed: "uFL"
